File: LMNC VCO - v1.2.sch (EAGLE design)
At the start: 49 parts, among them IC1 CEM3340, J1 JACKS, J10 LINK, P1 POWER, U1 TL072CP, U2 TL074CN

Commit message: Started Layout
Parts:
- added J2, J3, J4, J5, J6, J7, J8: PJ301_THONKICONNTME, og-pj301:PJ301_THONKICONNTME
- added R16: 10kB, parts_aman:POT_VERTICAL
- J1: value JACKS -> PJ301_THONKICONNTME; device con-headers-jp:F-1X10-SIP-100-32Y -> og-pj301:PJ301_THONKICONNTME; SPICEPREFIX X -> (none)
Connections:
- net 1VOCTIN: no longer J1.9
- net CVIN: no longer J1.8
- net FMINPUT: no longer J1.4
- net GND: no longer J1.1, J1.10
- net PWMIN: no longer J1.2
- net RAMPOUT: no longer J1.7
- net SQUAREOUT: no longer J1.3
- net SYNCIN1: no longer J1.6
- net TRIANGLEOUT: no longer J1.5

Commit message: up
Parts:
- removed R16: 10kB, parts_aman:POT_VERTICAL
- RV2: value 100K PWMLVL -> 100kB PWMLVL; device pot:EVUF2A -> parts_aman:POT_VERTICAL
- RV4: value 100K PW -> 100kB PW; device pot:EVUF2A -> parts_aman:POT_VERTICAL
- RV5: value 100K CV LVL -> 100kB CVLVL; device pot:EVUF2A -> parts_aman:POT_VERTICAL
- RV7: value 100K FINETUNE -> 100kB FINETUNE; device pot:EVUF2A -> parts_aman:POT_VERTICAL
Connections:
- net CVIN: now also RV5.B; no longer RV5.A
- net GND: now also RV5.A, RV7.B; no longer RV5.E, RV7.E
- net N$13: now also RV4.W; no longer RV4.S
- net N$14: now also RV2.W; no longer RV2.S
- net N$16: now also RV4.B; no longer RV4.E
- net N$22: now also RV7.W; no longer RV7.S
- net N$29: now also RV5.W; no longer RV5.S
- net PWMIN: now also RV2.B; no longer RV2.E
Other:
- moved on the sheet: R10, R20
